File: kicad/SevenSegmentModule/SevenSegmentModule.kicad_pcb (KiCad board)
At the start: 2 copper layers, 60.5 x 31.4 mm, 17 parts, among them J1 IN, J2 PIN, J4 OUT, J5 POUT, U2 Seven_Segment_With_Decimal

Commit message: Add modular PCBs and cleanup backups
Parts:
- removed TPIC6595: TPIC6595, Package_SO:SOIC-20W_7.5x12.8mm_P1.27mm
- added U1: TPIC6A595, Package_SO:SOIC-24W_7.5x15.4mm_P1.27mm, F.Cu at (165.8, 93.4)
- moved C1 6.79 mm to (168.3, 100.5)
Routing:
- net GND: track 11.1 -> 28.2 mm, vias 4 -> 8
- net Net-(U2-Pad4): track 5.95 -> 21.0 mm, vias 0 -> 1
- net Net-(U2-Pad12): track 22.3 -> 8.45 mm
- net Net-(U2-Pad2): track 5.42 -> 17.5 mm, vias 0 -> 1
- net Net-(U2-Pad10): track 17.3 -> 7.35 mm
- net Net-(U2-Pad6): track 6.47 -> 15.3 mm
- net Net-(U2-Pad14): track 26.2 -> 18.2 mm
- net Net-(U2-Pad8): track 7.67 -> 15.6 mm
- net SER_IN: track 29.8 -> 23.3 mm
- net Net-(U2-Pad16): track 28.5 -> 34.5 mm, vias 0 -> 2
- net G: track 60.9 -> 64.2 mm
- net SRCLR: track 57.8 -> 61.0 mm, vias 2 -> 3
- net SER_OUT: track 28.1 -> 25.8 mm
- net SRCK: track 57.6 -> 59.6 mm, vias 3 -> 2
- net RCLK: track 58.4 -> 57.5 mm
Other:
- board text added: "Seven Segment Module v1.1"
- board text removed: "SRCLK"
- board text removed: "Seven Segment Module v1.0"
